Commit message: perf: update urdf and meshes
- add field_link.stl
- decimate model files
- modify the colors

File: urdf/dart_system.urdf.xacro (robot description, xacro)
@@ -2,4 +2,16 @@
 <robot xmlns:xacro="http://www.ros.org/wiki/xacro"
   name="dart_system">
+  <material name="field_material">
+    <color rgba="0.4 0.4 0.4 1" />
+  </material>
+  <material name="aluminum">
+    <color rgba="0.65 0.68 0.72 1.0"/>
+  </material>
+  <material name="camera">
+    <color rgba="0.1 0.1 0.1 1.0"/>
+  </material>
+  <material name="base">
+    <color rgba="0.8 0.8 0.8 1.0"/>
+  </material>
   <!-- 基地现场偏差，均相对于 base_nominal_link 表达。默认值保持图纸位置不变。 -->
   <xacro:arg name="base_offset_x" default="0.0" />
@@ -13,14 +25,9 @@
   <link name="field_link">
     <!-- 薄板顶面与 field_link 的 z=0 平面重合。 -->
-    <visual name="field_area">
-      <origin
-        xyz="7.5 14.0 -0.005"
-        rpy="0.0 0.0 0.0" />
-      <geometry>
-        <box size="15.0 28.0 0.01" />
-      </geometry>
-      <material name="field_area_material">
-        <color rgba="0.3 0.3 0.3 1" />
-      </material>
+    <visual>
+      <geometry>
+        <mesh filename="package://dart_description/meshes/field_link.stl" scale="1 1 1"/>>
+      </geometry>
+      <material name="field_material"/>
     </visual>
   </link>
@@ -36,9 +43,7 @@
     <visual>
       <geometry>
-        <mesh filename="package://dart_description/meshes/base_link.STL" scale="1 1 1"/>
-      </geometry>
-      <material name="aluminum_material">
-        <color rgba="0.75 0.77 0.80 1.0" />
-      </material>
+        <mesh filename="package://dart_description/meshes/pnx_base_link.stl" scale="1 1 1"/>
+      </geometry>
+      <material name="base"/>
     </visual>
   </link>
@@ -61,6 +66,7 @@
     <visual>
       <geometry>
-        <mesh filename="package://dart_description/meshes/dart_detection_module_link.STL" scale="0.001 0.001 0.001"/>
-      </geometry>
+        <mesh filename="package://dart_description/meshes/pnx_dart_detection_module_link.stl" scale="1 1 1"/>
+      </geometry>
+      <material name="base"/>
     </visual>
   </link>
@@ -73,9 +79,19 @@
   </joint>
   <!-- 发光面直径约 55 mm，中心偏移与当前雷达定位配置保持一致。 -->
-  <link name="green_light_link"/>
+  <link name="green_light_link">
+    <visual>
+      <origin xyz="0.0 -0.004 0.0" rpy="${pi / 2} 0.0 0.0"/>
+      <geometry>
+        <cylinder radius="0.0275" length="0.01"/>
+      </geometry>
+      <material name="green_light_material">
+        <color rgba="0.2 1.0 0.2 1"/>
+      </material>
+    </visual>
+  </link>
   <joint name="dart_detection_module_to_green_light" type="fixed">
     <parent link="dart_detection_module_link" />
     <child link="green_light_link" />
-    <origin xyz="0.0 0.1222 0.02363" rpy="${pi / 9} 0.0 0.0" />
+    <origin xyz="0.0 0.1222 0.02363" rpy="${pi / 12} 0.0 0.0" />
   </joint>
   <!-- 装甲板模块，中心偏移与当前雷达定位配置保持一致。 -->
@@ -88,19 +104,9 @@
   <!-- 飞镖系统底座坐标系 -->
   <!-- 飞镖系统放置平面投影到底面中心 -->
-  <link name="dart_pedestal_link">
-    <visual name="dart_pedestal_area">
-      <origin xyz="0.0 0.0 0.1025" rpy="0.0 0.0 0.0" />
-      <geometry>
-        <box size="1.0 0.6 0.205" />
-      </geometry>
-      <material name="dart_pedestal_material">
-        <color rgba="0.498 0.498 0.498 1" />
-      </material>
-    </visual>
-  </link>
+  <link name="dart_pedestal_link"/>
   <joint name="field_to_dart_pedestal" type="fixed">
     <parent link="field_link" />
     <child link="dart_pedestal_link" />
-    <origin xyz="4.23 0.213 0.0" rpy="0.0 0.0 ${pi / 2}" />
+    <origin xyz="4.23 0.5 0.0" rpy="0.0 0.0 ${pi / 2}" />
   </joint>
   <!-- 镖架机械基准 -->
@@ -110,9 +116,7 @@
       <origin xyz="0.0 0.0 0.091" rpy="0.0 0.0 0.0" />
       <geometry>
-        <mesh filename="package://dart_description/meshes/dart_link.STL" scale="1 1 1" />
-      </geometry>
-      <material name="aluminum_material">
-        <color rgba="0.75 0.77 0.80 1.0" />
-      </material>
+        <mesh filename="package://dart_description/meshes/dart_base_link.stl" scale="1 1 1" />
+      </geometry>
+      <material name="aluminum"/>
     </visual>
   </link>
@@ -128,9 +132,7 @@
     <visual>
       <geometry>
-        <mesh filename="package://dart_description/meshes/launcher_frame.STL" scale="1 1 1" />
-      </geometry>
-      <material name="aluminum_material">
-        <color rgba="0.75 0.77 0.80 1.0" />
-      </material>
+        <mesh filename="package://dart_description/meshes/launcher_frame.stl" scale="1 1 1" />
+      </geometry>
+      <material name="aluminum"/>
     </visual>
   </link>
@@ -157,18 +159,14 @@
     <visual>
       <geometry>
-        <mesh filename="package://dart_description/meshes/MV-CA016-10UMUC.STL" scale="1 1 1" />
-      </geometry>
-      <material name="camera_material">
-        <color rgba="0.8 0.8 0.8 1" />
-      </material>
+        <mesh filename="package://dart_description/meshes/camera_mount_link_camera.stl" scale="1 1 1" />
+      </geometry>
+      <material name="camera"/>
     </visual>
     <visual>
       <origin xyz="0.012 0.0 0.015" rpy="0.0 0.0 0.0" />
       <geometry>
-        <mesh filename="package://dart_description/meshes/MVL-HF5028M-6MPE.STL" scale="1 1 1" />
-      </geometry>
-      <material name="camera_material">
-        <color rgba="0.8 0.8 0.8 1" />
-      </material>
+        <mesh filename="package://dart_description/meshes/camera_mount_link_lens.stl" scale="1 1 1" />
+      </geometry>
+      <material name="camera"/>
     </visual>
   </link>
@@ -192,9 +190,7 @@
     <visual>
       <geometry>
-        <mesh filename="package://dart_description/meshes/livox_lidar_Mid-70.STL" scale="1 1 1" />
-      </geometry>
-      <material name="livox_lidar_material">
-        <color rgba="0.85 0.87 0.90 1" />
-      </material>
+        <mesh filename="package://dart_description/meshes/lidar_mount_link.stl" scale="1 1 1" />
+      </geometry>
+      <material name="aluminum"/>
     </visual>
   </link>

Commit message: feat: add camera and lidar visualization

File: urdf/dart_system.urdf.xacro (robot description, xacro)
@@ -27,5 +27,5 @@
     <visual>
       <geometry>
-        <mesh filename="package://dart_description/meshes/field_link.stl" scale="1 1 1"/>>
+        <mesh filename="package://dart_description/meshes/field_link.stl" scale="1 1 1"/>
       </geometry>
       <material name="field_material"/>

Commit message: chore: update base and lidar position

File: urdf/dart_system.urdf.xacro (robot description, xacro)
@@ -37,5 +37,5 @@
     <parent link="field_link" />
     <child link="base_nominal_link" />
-    <origin xyz="7.5 25.593 0.0" rpy="0.0 0.0 ${pi}" />
+    <origin xyz="7.5 25.593 0.4" rpy="0.0 0.0 ${pi}" />
   </joint>
   <!-- 现场基地实际坐标系。偏差为零时与理论坐标系重合。 -->
@@ -198,5 +198,5 @@
     <parent link="launcher_frame" />
     <child link="lidar_mount_link" />
-    <origin xyz="0.35 0.0 0.42" rpy="0.0 0.0 0.0" />
+    <origin xyz="0.35 0.0 0.88" rpy="0.0 0.0 0.0" />
   </joint>
   <!-- 雷达测量坐标系 -->

Commit message: feat: change the parent link of lidar, modify the parameters

File: urdf/dart_system.urdf.xacro (robot description, xacro)
@@ -142,15 +142,8 @@
     <origin xyz="0.0 0.0 0.091" rpy="0.0 0.0 0.0" />
     <axis xyz="0 0 1" />
-    <limit lower="${-pi / 2}"
-      upper="${pi / 2}"
+    <limit lower="${-pi / 9}"
+      upper="0"
       effort="20"
       velocity="${10 * pi / 3}" />
-  </joint>
-  <!-- 飞镖释放坐标 -->
-  <link name="dart_release_frame" />
-  <joint name="launcher_to_dart_release" type="fixed">
-    <parent link="launcher_frame" />
-    <child link="dart_release_frame" />
-    <origin xyz="0.112 0.0 0.48" rpy="0.0 0.0 0.0" />
   </joint>
   <!-- 相机机械坐标 -->
@@ -174,5 +167,5 @@
     <parent link="launcher_frame" />
     <child link="camera_mount_link" />
-    <origin xyz="0.1 0.0 0.8" rpy="0.0 0.0 0.0" />
+    <origin xyz="0.1799 0.0 0.3164" rpy="0.0 0.0 ${-pi / 90}" />
   </joint>
   <!-- 相机光学坐标 -->
@@ -196,7 +189,7 @@
   </link>
   <joint name="launcher_to_lidar_mount" type="fixed">
-    <parent link="launcher_frame" />
+    <parent link="dart_base_link" />
     <child link="lidar_mount_link" />
-    <origin xyz="0.35 0.0 0.88" rpy="0.0 0.0 0.0" />
+    <origin xyz="0.3787 0.1718 0.484" rpy="0.0 0.0 ${-78 * pi / 1800}" />
   </joint>
   <!-- 雷达测量坐标系 -->

Commit message: chore: update parameters of base and lidar

File: urdf/dart_system.urdf.xacro (robot description, xacro)
@@ -37,5 +37,5 @@
     <parent link="field_link" />
     <child link="base_nominal_link" />
-    <origin xyz="7.5 25.593 0.4" rpy="0.0 0.0 ${pi}" />
+    <origin xyz="7.5 25.593 0.307" rpy="0.0 0.0 ${pi}" />
   </joint>
   <!-- 现场基地实际坐标系。偏差为零时与理论坐标系重合。 -->
@@ -114,5 +114,5 @@
   <link name="dart_base_link">
     <visual>
-      <origin xyz="0.0 0.0 0.091" rpy="0.0 0.0 0.0" />
+      <origin xyz="0.0 0.0 0.0" rpy="0.0 0.0 0.0" />
       <geometry>
         <mesh filename="package://dart_description/meshes/dart_base_link.stl" scale="1 1 1" />
@@ -191,5 +191,5 @@
     <parent link="dart_base_link" />
     <child link="lidar_mount_link" />
-    <origin xyz="0.3787 0.1718 0.484" rpy="0.0 0.0 ${-78 * pi / 1800}" />
+    <origin xyz="0.3787 0.1718 0.393" rpy="0.0 0.0 ${-78 * pi / 1800}" />
   </joint>
   <!-- 雷达测量坐标系 -->

Commit message: feat: add ground, door_roi and base_roi visualization

File: urdf/dart_system.urdf.xacro (robot description, xacro)
@@ -167,5 +167,5 @@
     <parent link="launcher_frame" />
     <child link="camera_mount_link" />
-    <origin xyz="0.1799 0.0 0.3164" rpy="0.0 0.0 ${-pi / 90}" />
+    <origin xyz="0.1799 0.0 0.3164" rpy="0.0 ${-pi / 90} 0.0" />
   </joint>
   <!-- 相机光学坐标 -->

Commit message: feat(stereo): change urdf to stereo, provide stereo visualization

File: urdf/dart_system.urdf.xacro (robot description, xacro)
@@ -78,5 +78,5 @@
     <limit lower="0.0" upper="0.56" effort="1.0" velocity="1.0" />
   </joint>
-  <!-- 发光面直径约 55 mm，中心偏移与当前雷达定位配置保持一致。 -->
+  <!-- 发光面直径约 55 mm，中心偏移沿用当前机构测量值。 -->
   <link name="green_light_link">
     <visual>
@@ -95,5 +95,5 @@
     <origin xyz="0.0 0.1222 0.02363" rpy="${pi / 12} 0.0 0.0" />
   </joint>
-  <!-- 装甲板模块，中心偏移与当前雷达定位配置保持一致。 -->
+  <!-- 装甲板模块，中心偏移沿用当前机构测量值。 -->
   <link name="armor_link"/>
   <joint name="dart_detection_module_to_armor" type="fixed">
@@ -147,12 +147,18 @@
       velocity="${10 * pi / 3}" />
   </joint>
-  <!-- 相机机械坐标 -->
-  <!-- 相机方形安装底面中心 -->
-  <link name="camera_mount_link">
+  <!-- 双相机固定板中心。左右相机的公共俯仰角在此处统一定义。 -->
+  <link name="stereo_camera_center_link" />
+  <joint name="launcher_to_stereo_camera_center" type="fixed">
+    <parent link="launcher_frame" />
+    <child link="stereo_camera_center_link" />
+    <origin xyz="0.1799 0.0 0.3164" rpy="0.0 ${-pi / 90} 0.0" />
+  </joint>
+  <!-- 左相机：相对双相机固定板中心向左 -->
+  <link name="left_camera_mount_link">
     <visual>
       <geometry>
         <mesh filename="package://dart_description/meshes/camera_mount_link_camera.stl" scale="1 1 1" />
       </geometry>
-      <material name="camera"/>
+      <material name="camera" />
     </visual>
     <visual>
@@ -161,42 +167,46 @@
         <mesh filename="package://dart_description/meshes/camera_mount_link_lens.stl" scale="1 1 1" />
       </geometry>
-      <material name="camera"/>
-    </visual>
-  </link>
-  <joint name="launcher_to_camera_mount" type="fixed">
-    <parent link="launcher_frame" />
-    <child link="camera_mount_link" />
-    <origin xyz="0.1799 0.0 0.3164" rpy="0.0 ${-pi / 90} 0.0" />
-  </joint>
-  <!-- 相机光学坐标 -->
-  <link name="camera_optical_frame" />
-  <joint name="camera_mount_to_optical" type="fixed">
-    <parent link="camera_mount_link" />
-    <child link="camera_optical_frame" />
-    <!-- camera_mount: x前 y左 z上
-         optical:      z前 x右 y下 -->
+      <material name="camera" />
+    </visual>
+  </link>
+  <joint name="stereo_camera_center_to_left_camera_mount" type="fixed">
+    <parent link="stereo_camera_center_link" />
+    <child link="left_camera_mount_link" />
+    <origin xyz="0.0 0.15 0.0" rpy="0.0 0.0 0.0" />
+  </joint>
+  <link name="left_camera_optical_frame" />
+  <joint name="left_camera_mount_to_optical" type="fixed">
+    <parent link="left_camera_mount_link" />
+    <child link="left_camera_optical_frame" />
+    <!-- mount: x前 y左 z上；optical: z前 x右 y下。 -->
     <origin xyz="0.04 0.0 0.015" rpy="${-pi / 2} 0.0 ${-pi / 2}" />
   </joint>
-  <!-- 雷达机械坐标
-       雷达安装底面中心 -->
-  <link name="lidar_mount_link">
-    <visual>
-      <geometry>
-        <mesh filename="package://dart_description/meshes/lidar_mount_link.stl" scale="1 1 1" />
-      </geometry>
-      <material name="aluminum"/>
-    </visual>
-  </link>
-  <joint name="launcher_to_lidar_mount" type="fixed">
-    <parent link="dart_base_link" />
-    <child link="lidar_mount_link" />
-    <origin xyz="0.3787 0.1718 0.393" rpy="0.0 0.0 ${-78 * pi / 1800}" />
-  </joint>
-  <!-- 雷达测量坐标系 -->
-  <link name="livox_frame" />
-  <joint name="lidar_mount_to_livox" type="fixed">
-    <parent link="lidar_mount_link" />
-    <child link="livox_frame" />
-    <origin xyz="0.0323 0.0 0.0324" rpy="0.0 0.0 0.0" />
+  <!-- 右相机：相对双相机固定板中心向右 -->
+  <link name="right_camera_mount_link">
+    <visual>
+      <geometry>
+        <mesh filename="package://dart_description/meshes/camera_mount_link_camera.stl" scale="1 1 1" />
+      </geometry>
+      <material name="camera" />
+    </visual>
+    <visual>
+      <origin xyz="0.012 0.0 0.015" rpy="0.0 0.0 0.0" />
+      <geometry>
+        <mesh filename="package://dart_description/meshes/camera_mount_link_lens.stl" scale="1 1 1" />
+      </geometry>
+      <material name="camera" />
+    </visual>
+  </link>
+  <joint name="stereo_camera_center_to_right_camera_mount" type="fixed">
+    <parent link="stereo_camera_center_link" />
+    <child link="right_camera_mount_link" />
+    <origin xyz="0.0 -0.15 0.0" rpy="0.0 0.0 0.0" />
+  </joint>
+  <link name="right_camera_optical_frame" />
+  <joint name="right_camera_mount_to_optical" type="fixed">
+    <parent link="right_camera_mount_link" />
+    <child link="right_camera_optical_frame" />
+    <!-- mount: x前 y左 z上；optical: z前 x右 y下。 -->
+    <origin xyz="0.04 0.0 0.015" rpy="${-pi / 2} 0.0 ${-pi / 2}" />
   </joint>
 </robot>

Commit message: chore: update models, camera parameters and urdf

File: urdf/dart_system.urdf.xacro (robot description, xacro)
@@ -148,9 +148,16 @@
   </joint>
   <!-- 双相机固定板中心。左右相机的公共俯仰角在此处统一定义。 -->
-  <link name="stereo_camera_center_link" />
+  <link name="stereo_camera_center_link" >
+    <visual>
+      <geometry>
+        <mesh filename="package://dart_description/meshes/stereo_camera_center_link.stl" scale="1 1 1"/>
+      </geometry>
+      <material name="aluminum" />
+    </visual>
+  </link>
   <joint name="launcher_to_stereo_camera_center" type="fixed">
     <parent link="launcher_frame" />
     <child link="stereo_camera_center_link" />
-    <origin xyz="0.1799 0.0 0.3164" rpy="0.0 ${-pi / 90} 0.0" />
+    <origin xyz="0.19 0.0 0.308" rpy="0.0 0.0 0.0" />
   </joint>
   <!-- 左相机：相对双相机固定板中心向左 -->
@@ -173,5 +180,5 @@
     <parent link="stereo_camera_center_link" />
     <child link="left_camera_mount_link" />
-    <origin xyz="0.0 0.15 0.0" rpy="0.0 0.0 0.0" />
+    <origin xyz="-0.015 0.15 0.0" rpy="0.0 0.0 0.0" />
   </joint>
   <link name="left_camera_optical_frame" />
@@ -201,5 +208,5 @@
     <parent link="stereo_camera_center_link" />
     <child link="right_camera_mount_link" />
-    <origin xyz="0.0 -0.15 0.0" rpy="0.0 0.0 0.0" />
+    <origin xyz="-0.015 -0.15 0.0" rpy="0.0 0.0 0.0" />
   </joint>
   <link name="right_camera_optical_frame" />

Commit message: feat(urdf): change the parent link of right_camera_mount_link to left_camera_mount_link

File: urdf/dart_system.urdf.xacro (robot description, xacro)
@@ -206,7 +206,7 @@
   </link>
   <joint name="stereo_camera_center_to_right_camera_mount" type="fixed">
-    <parent link="stereo_camera_center_link" />
+    <parent link="left_camera_mount_link" />
     <child link="right_camera_mount_link" />
-    <origin xyz="-0.015 -0.15 0.0" rpy="0.0 0.0 0.0" />
+    <origin xyz="0.0 -0.3 0.0" rpy="0.0 0.0 0.0" />
   </joint>
   <link name="right_camera_optical_frame" />

Commit message: feat: update stereo camera position

File: urdf/dart_system.urdf.xacro (robot description, xacro)
@@ -148,16 +148,9 @@
   </joint>
   <!-- 双相机固定板中心。左右相机的公共俯仰角在此处统一定义。 -->
-  <link name="stereo_camera_center_link" >
-    <visual>
-      <geometry>
-        <mesh filename="package://dart_description/meshes/stereo_camera_center_link.stl" scale="1 1 1"/>
-      </geometry>
-      <material name="aluminum" />
-    </visual>
-  </link>
+  <link name="stereo_camera_center_link" />
   <joint name="launcher_to_stereo_camera_center" type="fixed">
     <parent link="launcher_frame" />
     <child link="stereo_camera_center_link" />
-    <origin xyz="0.19 0.0 0.308" rpy="0.0 0.0 0.0" />
+    <origin xyz="0.23658 0.0 0.42645" rpy="0.0 0.0 0.0" />
   </joint>
   <!-- 左相机：相对双相机固定板中心向左 -->
@@ -180,5 +173,5 @@
     <parent link="stereo_camera_center_link" />
     <child link="left_camera_mount_link" />
-    <origin xyz="-0.015 0.15 0.0" rpy="0.0 0.0 0.0" />
+    <origin xyz="0.0 0.13 0.0" rpy="${-pi / 2} 0.0 0.0" />
   </joint>
   <link name="left_camera_optical_frame" />
@@ -208,5 +201,5 @@
     <parent link="stereo_camera_center_link" />
     <child link="right_camera_mount_link" />
-    <origin xyz="-0.015 -0.15 0.0" rpy="0.0 0.0 0.0" />
+    <origin xyz="0.0 -0.13 0.0" rpy="${pi / 2} 0.0 0.0" />
   </joint>
   <link name="right_camera_optical_frame" />

Commit message: fix: center detection module slide range at zero

File: urdf/dart_system.urdf.xacro (robot description, xacro)
@@ -55,10 +55,10 @@
       rpy="$(arg base_offset_roll) $(arg base_offset_pitch) $(arg base_offset_yaw)" />
   </joint>
-  <!-- 滑轨零位，默认在基地左侧 -->
+  <!-- 滑轨零位位于行程中心 -->
   <link name="rail_origin_link" />
   <joint name="base_to_rail_origin" type="fixed">
     <parent link="base_link" />
     <child link="rail_origin_link" />
-    <origin xyz="-0.28 -0.03193 0.91" rpy="0.0 0.0 0.0" />
+    <origin xyz="0.0 -0.03193 0.91" rpy="0.0 0.0 0.0" />
   </joint>
   <!-- 飞镖检测模块运动位置 -->
@@ -76,5 +76,5 @@
     <origin xyz="0.0 0.0 0.0" rpy="0.0 0.0 0.0" />
     <axis xyz="1 0 0" />
-    <limit lower="0.0" upper="0.56" effort="1.0" velocity="1.0" />
+    <limit lower="-0.28" upper="0.28" effort="1.0" velocity="1.0" />
   </joint>
   <!-- 发光面直径约 55 mm，中心偏移沿用当前机构测量值。 -->
