Commit message: feat: model launcher and target impact geometry
Define release and armor surface frames, align the detection module
geometry, and expose reusable URDF-based kinematics for impact analysis.

File: urdf/dart_system.urdf.xacro (robot description, xacro)
@@ -6,11 +6,11 @@
   </material>
   <material name="aluminum">
-    <color rgba="0.65 0.68 0.72 1.0"/>
+    <color rgba="0.65 0.68 0.72 1.0" />
   </material>
   <material name="camera">
-    <color rgba="0.1 0.1 0.1 1.0"/>
+    <color rgba="0.1 0.1 0.1 1.0" />
   </material>
   <material name="base">
-    <color rgba="0.8 0.8 0.8 1.0"/>
+    <color rgba="0.8 0.8 0.8 1.0" />
   </material>
   <!-- 基地现场偏差，均相对于 base_nominal_link 表达。默认值保持图纸位置不变。 -->
@@ -21,4 +21,20 @@
   <xacro:arg name="base_offset_pitch" default="0.0" />
   <xacro:arg name="base_offset_yaw" default="0.0" />
+  <!--
+    飞镖离开导轨时的参考点与初始方向，均相对于 launcher_frame 表达。
+    dart_release_link 的 +x 沿飞镖初始发射方向；负 pitch 对应向上的发射仰角。
+  -->
+  <xacro:arg name="dart_release_x" default="0.2" />
+  <xacro:arg name="dart_release_y" default="0.0" />
+  <xacro:arg name="dart_release_z" default="0.6" />
+  <xacro:arg name="dart_release_pitch" default="${-32 * pi / 180}" />
+  <!--
+    armor_link 位于装甲板上表面中心，实体沿 local -x 延伸。
+    local y/z 张成上表面，local +x 为上表面法向。
+    box 的 armor_size_x 方向经 visual/collision 旋转后对应 armor_link local z。
+  -->
+  <xacro:arg name="armor_size_x" default="0.1" />
+  <xacro:arg name="armor_size_y" default="0.1" />
+  <xacro:arg name="armor_thickness" default="0.01" />
   <!-- 场地坐标系：x 右、y 前、z 上 -->
   <!-- 以场地左下角为原点 -->
@@ -27,7 +43,7 @@
     <visual>
       <geometry>
-        <mesh filename="package://dart_description/meshes/field_link.stl" scale="1 1 1"/>
-      </geometry>
-      <material name="field_material"/>
+        <mesh filename="package://dart_description/meshes/field_link.stl" scale="1 1 1" />
+      </geometry>
+      <material name="field_material" />
     </visual>
   </link>
@@ -37,5 +53,5 @@
     <parent link="field_link" />
     <child link="base_nominal_link" />
-    <origin xyz="7.5 25.593 0.307" rpy="0.0 0.0 ${pi}" />
+    <origin xyz="7.5 25.593 0.307" rpy="0.0 0.0 ${-pi / 2}" />
   </joint>
   <!-- 现场基地实际坐标系。偏差为零时与理论坐标系重合。 -->
@@ -43,7 +59,7 @@
     <visual>
       <geometry>
-        <mesh filename="package://dart_description/meshes/pnx_base_link.stl" scale="1 1 1"/>
-      </geometry>
-      <material name="base"/>
+        <mesh filename="package://dart_description/meshes/pnx_base_link.stl" scale="1 1 1" />
+      </geometry>
+      <material name="base" />
     </visual>
   </link>
@@ -60,5 +76,5 @@
     <parent link="base_link" />
     <child link="rail_origin_link" />
-    <origin xyz="0.0 -0.03193 0.91" rpy="0.0 0.0 0.0" />
+    <origin xyz="-0.03193 0.0 0.91" rpy="0.0 0.0 0.0" />
   </joint>
   <!-- 飞镖检测模块运动位置 -->
@@ -66,7 +82,8 @@
     <visual>
       <geometry>
-        <mesh filename="package://dart_description/meshes/pnx_dart_detection_module_link.stl" scale="1 1 1"/>
-      </geometry>
-      <material name="base"/>
+        <mesh filename="package://dart_description/meshes/pnx_dart_detection_module_link.stl"
+          scale="1 1 1" />
+      </geometry>
+      <material name="base" />
     </visual>
   </link>
@@ -75,5 +92,5 @@
     <child link="dart_detection_module_link" />
     <origin xyz="0.0 0.0 0.0" rpy="0.0 0.0 0.0" />
-    <axis xyz="1 0 0" />
+    <axis xyz="0 1 0" />
     <limit lower="-0.28" upper="0.28" effort="1.0" velocity="1.0" />
   </joint>
@@ -81,10 +98,10 @@
   <link name="green_light_link">
     <visual>
-      <origin xyz="0.0 -0.004 0.0" rpy="${pi / 2} 0.0 0.0"/>
-      <geometry>
-        <cylinder radius="0.0275" length="0.01"/>
+      <origin xyz="-0.0049 0.0 0.0" rpy="0.0 ${-pi / 2} 0.0" />
+      <geometry>
+        <cylinder radius="0.0275" length="0.01" />
       </geometry>
       <material name="green_light_material">
-        <color rgba="0.2 1.0 0.2 1"/>
+        <color rgba="0.2 1.0 0.2 1" />
       </material>
     </visual>
@@ -93,16 +110,30 @@
     <parent link="dart_detection_module_link" />
     <child link="green_light_link" />
-    <origin xyz="0.0 0.1222 0.02363" rpy="${pi / 12} 0.0 0.0" />
-  </joint>
-  <!-- 装甲板模块，中心偏移沿用当前机构测量值。 -->
-  <link name="armor_link"/>
+    <origin xyz="0.1222 0.0 0.02363" rpy="0.0 ${-14.5 * pi / 180} 0.0" />
+  </joint>
+  <!-- 装甲板模块；armor_link 原点为装甲板上表面中心。 -->
+  <link name="armor_link">
+    <visual>
+      <origin xyz="${-float(xacro.arg('armor_thickness')) / 2 + 0.0001} 0.0 0.0" rpy="0.0 ${pi / 2} 0.0" />
+      <geometry>
+        <box size="$(arg armor_size_x) $(arg armor_size_y) $(arg armor_thickness)" />
+      </geometry>
+      <material name="aluminum" />
+    </visual>
+    <collision>
+      <origin xyz="${-float(xacro.arg('armor_thickness')) / 2} 0.0 0.0" rpy="0.0 ${pi / 2} 0.0" />
+      <geometry>
+        <box size="$(arg armor_size_x) $(arg armor_size_y) $(arg armor_thickness)" />
+      </geometry>
+    </collision>
+  </link>
   <joint name="dart_detection_module_to_armor" type="fixed">
     <parent link="dart_detection_module_link" />
     <child link="armor_link" />
-    <origin xyz="0.0 0.05384 0.10249" rpy="${pi / 3} 0.0 0.0" />
+    <origin xyz="0.05384 0.0 0.10249" rpy="0.0 ${-62.5 * pi / 180} 0.0" />
   </joint>
   <!-- 飞镖系统底座坐标系 -->
   <!-- 飞镖系统放置平面投影到底面中心 -->
-  <link name="dart_pedestal_link"/>
+  <link name="dart_pedestal_link" />
   <joint name="field_to_dart_pedestal" type="fixed">
     <parent link="field_link" />
@@ -118,5 +149,5 @@
         <mesh filename="package://dart_description/meshes/dart_base_link.stl" scale="1 1 1" />
       </geometry>
-      <material name="aluminum"/>
+      <material name="aluminum" />
     </visual>
   </link>
@@ -134,5 +165,5 @@
         <mesh filename="package://dart_description/meshes/launcher_frame.stl" scale="1 1 1" />
       </geometry>
-      <material name="aluminum"/>
+      <material name="aluminum" />
     </visual>
   </link>
@@ -147,4 +178,13 @@
       velocity="${10 * pi / 3}" />
   </joint>
+  <!-- 飞镖离轨点；local +x 为固定发射方向。 -->
+  <link name="dart_release_link" />
+  <joint name="launcher_to_dart_release" type="fixed">
+    <parent link="launcher_frame" />
+    <child link="dart_release_link" />
+    <origin
+      xyz="$(arg dart_release_x) $(arg dart_release_y) $(arg dart_release_z)"
+      rpy="0.0 $(arg dart_release_pitch) 0.0" />
+  </joint>
   <!-- 双相机固定板中心。左右相机的公共俯仰角在此处统一定义。 -->
   <link name="stereo_camera_center_link" />
@@ -158,5 +198,6 @@
     <visual>
       <geometry>
-        <mesh filename="package://dart_description/meshes/camera_mount_link_camera.stl" scale="1 1 1" />
+        <mesh filename="package://dart_description/meshes/camera_mount_link_camera.stl"
+          scale="1 1 1" />
       </geometry>
       <material name="camera" />
@@ -186,5 +227,6 @@
     <visual>
       <geometry>
-        <mesh filename="package://dart_description/meshes/camera_mount_link_camera.stl" scale="1 1 1" />
+        <mesh filename="package://dart_description/meshes/camera_mount_link_camera.stl"
+          scale="1 1 1" />
       </geometry>
       <material name="camera" />

Commit message: feat: add the RM2027 scene and standalone rig mode
- Replace legacy field assets with shared colored CAD meshes.
- Separate runtime rig transforms from full-scene visualization.
- Correct target surfaces, mounting datums, and gate motion.
- Organize offline tools and metadata, and validate geometry APIs.

File: urdf/dart_system.urdf.xacro (robot description, xacro)
@@ -1,254 +1,13 @@
-<?xml version="1.0"?>
-<robot xmlns:xacro="http://www.ros.org/wiki/xacro"
-  name="dart_system">
-  <material name="field_material">
-    <color rgba="0.4 0.4 0.4 1" />
-  </material>
-  <material name="aluminum">
-    <color rgba="0.65 0.68 0.72 1.0" />
-  </material>
-  <material name="camera">
-    <color rgba="0.1 0.1 0.1 1.0" />
-  </material>
-  <material name="base">
-    <color rgba="0.8 0.8 0.8 1.0" />
-  </material>
-  <!-- 基地现场偏差，均相对于 base_nominal_link 表达。默认值保持图纸位置不变。 -->
-  <xacro:arg name="base_offset_x" default="0.0" />
-  <xacro:arg name="base_offset_y" default="0.0" />
-  <xacro:arg name="base_offset_z" default="0.0" />
-  <xacro:arg name="base_offset_roll" default="0.0" />
-  <xacro:arg name="base_offset_pitch" default="0.0" />
-  <xacro:arg name="base_offset_yaw" default="0.0" />
-  <!--
-    飞镖离开导轨时的参考点与初始方向，均相对于 launcher_frame 表达。
-    dart_release_link 的 +x 沿飞镖初始发射方向；负 pitch 对应向上的发射仰角。
-  -->
-  <xacro:arg name="dart_release_x" default="0.2" />
-  <xacro:arg name="dart_release_y" default="0.0" />
-  <xacro:arg name="dart_release_z" default="0.6" />
-  <xacro:arg name="dart_release_pitch" default="${-32 * pi / 180}" />
-  <!--
-    armor_link 位于装甲板上表面中心，实体沿 local -x 延伸。
-    local y/z 张成上表面，local +x 为上表面法向。
-    box 的 armor_size_x 方向经 visual/collision 旋转后对应 armor_link local z。
-  -->
-  <xacro:arg name="armor_size_x" default="0.1" />
-  <xacro:arg name="armor_size_y" default="0.1" />
-  <xacro:arg name="armor_thickness" default="0.01" />
-  <!-- 场地坐标系：x 右、y 前、z 上 -->
-  <!-- 以场地左下角为原点 -->
-  <link name="field_link">
-    <!-- 薄板顶面与 field_link 的 z=0 平面重合。 -->
-    <visual>
-      <geometry>
-        <mesh filename="package://dart_description/meshes/field_link.stl" scale="1 1 1" />
-      </geometry>
-      <material name="field_material" />
-    </visual>
-  </link>
-  <!-- 图纸中的基地理论坐标系。该变换不由现场标定修改。 -->
-  <link name="base_nominal_link" />
-  <joint name="field_to_base_nominal" type="fixed">
-    <parent link="field_link" />
-    <child link="base_nominal_link" />
-    <origin xyz="7.5 25.593 0.307" rpy="0.0 0.0 ${-pi / 2}" />
-  </joint>
-  <!-- 现场基地实际坐标系。偏差为零时与理论坐标系重合。 -->
-  <link name="base_link">
-    <visual>
-      <geometry>
-        <mesh filename="package://dart_description/meshes/pnx_base_link.stl" scale="1 1 1" />
-      </geometry>
-      <material name="base" />
-    </visual>
-  </link>
-  <joint name="base_nominal_to_base" type="fixed">
-    <parent link="base_nominal_link" />
-    <child link="base_link" />
-    <origin
-      xyz="$(arg base_offset_x) $(arg base_offset_y) $(arg base_offset_z)"
-      rpy="$(arg base_offset_roll) $(arg base_offset_pitch) $(arg base_offset_yaw)" />
-  </joint>
-  <!-- 滑轨零位位于行程中心 -->
-  <link name="rail_origin_link" />
-  <joint name="base_to_rail_origin" type="fixed">
-    <parent link="base_link" />
-    <child link="rail_origin_link" />
-    <origin xyz="-0.03193 0.0 0.91" rpy="0.0 0.0 0.0" />
-  </joint>
-  <!-- 飞镖检测模块运动位置 -->
-  <link name="dart_detection_module_link">
-    <visual>
-      <geometry>
-        <mesh filename="package://dart_description/meshes/pnx_dart_detection_module_link.stl"
-          scale="1 1 1" />
-      </geometry>
-      <material name="base" />
-    </visual>
-  </link>
-  <joint name="dart_detection_module_slide_joint" type="prismatic">
-    <parent link="rail_origin_link" />
-    <child link="dart_detection_module_link" />
-    <origin xyz="0.0 0.0 0.0" rpy="0.0 0.0 0.0" />
-    <axis xyz="0 1 0" />
-    <limit lower="-0.28" upper="0.28" effort="1.0" velocity="1.0" />
-  </joint>
-  <!-- 发光面直径约 55 mm，中心偏移沿用当前机构测量值。 -->
-  <link name="green_light_link">
-    <visual>
-      <origin xyz="-0.0049 0.0 0.0" rpy="0.0 ${-pi / 2} 0.0" />
-      <geometry>
-        <cylinder radius="0.0275" length="0.01" />
-      </geometry>
-      <material name="green_light_material">
-        <color rgba="0.2 1.0 0.2 1" />
-      </material>
-    </visual>
-  </link>
-  <joint name="dart_detection_module_to_green_light" type="fixed">
-    <parent link="dart_detection_module_link" />
-    <child link="green_light_link" />
-    <origin xyz="0.1222 0.0 0.02363" rpy="0.0 ${-14.5 * pi / 180} 0.0" />
-  </joint>
-  <!-- 装甲板模块；armor_link 原点为装甲板上表面中心。 -->
-  <link name="armor_link">
-    <visual>
-      <origin xyz="${-float(xacro.arg('armor_thickness')) / 2 + 0.0001} 0.0 0.0" rpy="0.0 ${pi / 2} 0.0" />
-      <geometry>
-        <box size="$(arg armor_size_x) $(arg armor_size_y) $(arg armor_thickness)" />
-      </geometry>
-      <material name="aluminum" />
-    </visual>
-    <collision>
-      <origin xyz="${-float(xacro.arg('armor_thickness')) / 2} 0.0 0.0" rpy="0.0 ${pi / 2} 0.0" />
-      <geometry>
-        <box size="$(arg armor_size_x) $(arg armor_size_y) $(arg armor_thickness)" />
-      </geometry>
-    </collision>
-  </link>
-  <joint name="dart_detection_module_to_armor" type="fixed">
-    <parent link="dart_detection_module_link" />
-    <child link="armor_link" />
-    <origin xyz="0.05384 0.0 0.10249" rpy="0.0 ${-62.5 * pi / 180} 0.0" />
-  </joint>
-  <!-- 飞镖系统底座坐标系 -->
-  <!-- 飞镖系统放置平面投影到底面中心 -->
-  <link name="dart_pedestal_link" />
-  <joint name="field_to_dart_pedestal" type="fixed">
-    <parent link="field_link" />
-    <child link="dart_pedestal_link" />
-    <origin xyz="4.23 0.5 0.0" rpy="0.0 0.0 ${pi / 2}" />
-  </joint>
-  <!-- 镖架机械基准 -->
-  <!-- 发射机构旋转轴与飞镖系统放置平面交点 -->
-  <link name="dart_base_link">
-    <visual>
-      <origin xyz="0.0 0.0 0.0" rpy="0.0 0.0 0.0" />
-      <geometry>
-        <mesh filename="package://dart_description/meshes/dart_base_link.stl" scale="1 1 1" />
-      </geometry>
-      <material name="aluminum" />
-    </visual>
-  </link>
-  <joint name="dart_pedestal_to_base" type="fixed">
-    <parent link="dart_pedestal_link" />
-    <child link="dart_base_link" />
-    <origin
-      xyz="0.0 0.0 0.205" rpy="0.0 0.0 0.0" />
-  </joint>
-  <!-- 发射机构方向 -->
-  <!-- 电机上方转盘中心 -->
-  <link name="launcher_frame">
-    <visual>
-      <geometry>
-        <mesh filename="package://dart_description/meshes/launcher_frame.stl" scale="1 1 1" />
-      </geometry>
-      <material name="aluminum" />
-    </visual>
-  </link>
-  <joint name="launcher_yaw_joint" type="revolute">
-    <parent link="dart_base_link" />
-    <child link="launcher_frame" />
-    <origin xyz="0.0 0.0 0.091" rpy="0.0 0.0 0.0" />
-    <axis xyz="0 0 1" />
-    <limit lower="${-pi / 9}"
-      upper="0"
-      effort="20"
-      velocity="${10 * pi / 3}" />
-  </joint>
-  <!-- 飞镖离轨点；local +x 为固定发射方向。 -->
-  <link name="dart_release_link" />
-  <joint name="launcher_to_dart_release" type="fixed">
-    <parent link="launcher_frame" />
-    <child link="dart_release_link" />
-    <origin
-      xyz="$(arg dart_release_x) $(arg dart_release_y) $(arg dart_release_z)"
-      rpy="0.0 $(arg dart_release_pitch) 0.0" />
-  </joint>
-  <!-- 双相机固定板中心。左右相机的公共俯仰角在此处统一定义。 -->
-  <link name="stereo_camera_center_link" />
-  <joint name="launcher_to_stereo_camera_center" type="fixed">
-    <parent link="launcher_frame" />
-    <child link="stereo_camera_center_link" />
-    <origin xyz="0.23658 0.0 0.42645" rpy="0.0 0.0 0.0" />
-  </joint>
-  <!-- 左相机：相对双相机固定板中心向左 -->
-  <link name="left_camera_mount_link">
-    <visual>
-      <geometry>
-        <mesh filename="package://dart_description/meshes/camera_mount_link_camera.stl"
-          scale="1 1 1" />
-      </geometry>
-      <material name="camera" />
-    </visual>
-    <visual>
-      <origin xyz="0.012 0.0 0.015" rpy="0.0 0.0 0.0" />
-      <geometry>
-        <mesh filename="package://dart_description/meshes/camera_mount_link_lens.stl" scale="1 1 1" />
-      </geometry>
-      <material name="camera" />
-    </visual>
-  </link>
-  <joint name="stereo_camera_center_to_left_camera_mount" type="fixed">
-    <parent link="stereo_camera_center_link" />
-    <child link="left_camera_mount_link" />
-    <origin xyz="0.0 0.13 0.0" rpy="${-pi / 2} 0.0 0.0" />
-  </joint>
-  <link name="left_camera_optical_frame" />
-  <joint name="left_camera_mount_to_optical" type="fixed">
-    <parent link="left_camera_mount_link" />
-    <child link="left_camera_optical_frame" />
-    <!-- mount: x前 y左 z上；optical: z前 x右 y下。 -->
-    <origin xyz="0.04 0.0 0.015" rpy="${-pi / 2} 0.0 ${-pi / 2}" />
-  </joint>
-  <!-- 右相机：相对双相机固定板中心向右 -->
-  <link name="right_camera_mount_link">
-    <visual>
-      <geometry>
-        <mesh filename="package://dart_description/meshes/camera_mount_link_camera.stl"
-          scale="1 1 1" />
-      </geometry>
-      <material name="camera" />
-    </visual>
-    <visual>
-      <origin xyz="0.012 0.0 0.015" rpy="0.0 0.0 0.0" />
-      <geometry>
-        <mesh filename="package://dart_description/meshes/camera_mount_link_lens.stl" scale="1 1 1" />
-      </geometry>
-      <material name="camera" />
-    </visual>
-  </link>
-  <joint name="stereo_camera_center_to_right_camera_mount" type="fixed">
-    <parent link="stereo_camera_center_link" />
-    <child link="right_camera_mount_link" />
-    <origin xyz="0.0 -0.13 0.0" rpy="${pi / 2} 0.0 0.0" />
-  </joint>
-  <link name="right_camera_optical_frame" />
-  <joint name="right_camera_mount_to_optical" type="fixed">
-    <parent link="right_camera_mount_link" />
-    <child link="right_camera_optical_frame" />
-    <!-- mount: x前 y左 z上；optical: z前 x右 y下。 -->
-    <origin xyz="0.04 0.0 0.015" rpy="${-pi / 2} 0.0 ${-pi / 2}" />
-  </joint>
+<?xml version='1.0' encoding='utf-8'?>
+<robot xmlns:xacro="http://www.ros.org/wiki/xacro" name="dart_system">
+  <xacro:include filename="modules/materials.xacro" />
+  <xacro:arg name="team" default="red" />
+  <xacro:property name="team" value="$(arg team)" />
+  <xacro:include filename="modules/field.xacro" />
+  <xacro:include filename="modules/bases.xacro" />
+  <xacro:include filename="modules/outposts.xacro" />
+  <xacro:include filename="modules/dart_stations.xacro" />
+  <xacro:include filename="modules/targets.xacro" />
+  <xacro:include filename="modules/launcher.xacro" />
+  <xacro:include filename="modules/stereo_camera.xacro" />
 </robot>
