Commit message: chore: update stereo camera position

File: urdf/modules/stereo_camera.xacro (robot description, xacro)
@@ -5,5 +5,5 @@
     <parent link="launcher_frame" />
     <child link="stereo_camera_center_link" />
-    <origin xyz="0.23658 0.0 0.42645" rpy="0.0 0.0 0.0" />
+    <origin xyz="0.2 0.0 0.383" rpy="0.0 0.0 0.0" />
   </joint>
   <link name="left_camera_mount_link">
@@ -25,5 +25,5 @@
     <parent link="stereo_camera_center_link" />
     <child link="left_camera_mount_link" />
-    <origin xyz="0.0 0.13 0.0" rpy="${-pi / 2} 0.0 0.0" />
+    <origin xyz="0.0 0.075 0.0" rpy="${-pi / 2} ${-pi / 90} 0.0" />
   </joint>
   <link name="left_camera_optical_frame" />
@@ -51,5 +51,5 @@
     <parent link="stereo_camera_center_link" />
     <child link="right_camera_mount_link" />
-    <origin xyz="0.0 -0.13 0.0" rpy="${pi / 2} 0.0 0.0" />
+    <origin xyz="0.0 -0.075 0.0" rpy="${pi / 2} ${-pi / 90} 0.0" />
   </joint>
   <link name="right_camera_optical_frame" />
